Commit message: tf stuff

File: config/urdf/version_6/arm_v2.xacro (robot description, xacro)
@@ -5,9 +5,22 @@
         <color rgba="0.7 0.7 0.7 1.0" />
     </material>
-    <joint name="arm_segment_0_joint" type="continuous">
+    <joint name="arm_base_joint" type="fixed">
         <parent link="chassis"/>
+        <child link="arm_base_link"/>
+        <origin xyz="0.15 0 0.0445" rpy="${pi/2} 0 0"/>
+    </joint>
+    <link name="arm_base_link">
+        <inertial>
+            <origin xyz="0 0 0" rpy="0 0 0"/>
+            <mass value="0.1"/>
+            <inertia ixx="0.01" ixy="0.0" ixz="0.0" iyy="0.01" iyz="0.0" izz="0.01"/>
+        </inertial>
+    </link>
+    <joint name="arm_segment_0_joint" type="revolute">
+        <parent link="arm_base_link"/>
         <child link="arm_segment_0"/>
-        <origin xyz="0.15 0 0.0445" rpy="${pi/2} 0 0"/>
+        <origin xyz="0 0 0" rpy="0 0 0"/>
         <axis xyz="0 0 1" />
+        <limit lower="0" upper="0" velocity="0" effort="0"/>
     </joint>
     <link name="arm_segment_0">
@@ -25,9 +38,10 @@
         </visual>
     </link>
-    <joint name="arm_segment_1_joint" type="continuous">
+    <joint name="arm_segment_1_joint" type="revolute">
         <parent link="arm_segment_0"/>
         <child link="arm_segment_1"/>
         <origin xyz="-0.1 0 0" rpy="0 0 0"/>
         <axis xyz="0 0 1" />
+        <limit lower="0" upper="0" velocity="0" effort="0"/>
     </joint>
     <link name="arm_segment_1">
@@ -45,9 +59,10 @@
         </visual>
     </link>
-    <joint name="arm_segment_2_joint" type="continuous">
+    <joint name="arm_segment_2_joint" type="revolute">
         <parent link="arm_segment_1"/>
         <child link="arm_segment_2"/>
         <origin xyz="-0.02 0.05 0" rpy="0 0 0"/>
         <axis xyz="0 0 1" />
+        <limit lower="0" upper="0" velocity="0" effort="0"/>
     </joint>
     <link name="arm_segment_2">

File: config/urdf/version_6/gripper.xacro (robot description, xacro)
@@ -14,11 +14,24 @@
         <origin xyz="0.022 -0.0255 0.0225" rpy="0 0 0"/>
     </xacro:sensor_d435>
-    <joint name="gripper_joint" type="continuous">
+    <joint name="gripper_joint" type="revolute">
         <parent link="gripper_base" />
         <child link="gripper_link" />
         <origin xyz="-0.0207 0.0125 0.0355" rpy="0 0 0"/>
         <axis xyz="0 0 1" />
+        <limit lower="0" upper="0" velocity="0" effort="0"/>
     </joint>
     <link name="gripper_link">
+        <inertial>
+            <origin xyz="0 0 0" rpy="0 0 0"/>
+            <mass value="0.1"/>
+            <inertia ixx="0.01" ixy="0.0" ixz="0.0" iyy="0.01" iyz="0.0" izz="0.01"/>
+        </inertial>
+    </link>
+    <joint name="arm_end_effector_joint" type="fixed">
+        <parent link="gripper_base" />
+        <child link="arm_end_effector" />
+        <origin xyz="0.1 -0.0002 0" rpy="${pi/2} 0 0"/>
+    </joint>
+    <link name="arm_end_effector">
         <inertial>
             <origin xyz="0 0 0" rpy="0 0 0"/>

Commit message: arm controller

File: config/urdf/version_6/arm_v2.xacro (robot description, xacro)
@@ -22,5 +22,5 @@
         <origin xyz="0 0 0" rpy="0 0 0"/>
         <axis xyz="0 0 1" />
-        <limit lower="0" upper="0" velocity="0" effort="0"/>
+        <limit lower="-3.826" upper="0" velocity="0" effort="0"/>
     </joint>
     <link name="arm_segment_0">
@@ -43,5 +43,5 @@
         <origin xyz="-0.1 0 0" rpy="0 0 0"/>
         <axis xyz="0 0 1" />
-        <limit lower="0" upper="0" velocity="0" effort="0"/>
+        <limit lower="-0.785398163" upper="1.570796327" velocity="0" effort="0"/>
     </joint>
     <link name="arm_segment_1">
@@ -64,5 +64,5 @@
         <origin xyz="-0.02 0.05 0" rpy="0 0 0"/>
         <axis xyz="0 0 1" />
-        <limit lower="0" upper="0" velocity="0" effort="0"/>
+        <limit lower="0" upper="3.091592654" velocity="0" effort="0"/>
     </joint>
     <link name="arm_segment_2">

Commit message: model in simulation

File: config/urdf/version_6/arm_v2.xacro (robot description, xacro)
@@ -27,15 +27,13 @@
         </xacro:inertial_box>
         <collision>
-            <origin xyz="0 0 0" rpy="${-pi/2} 0 0"/>
+            <!-- <origin xyz="0 0 0" rpy="${-pi/2} 0 0"/>
             <geometry>
                 <mesh filename="${mesh_folder}version_6/arm_v2/arm_segment_0_reduced.stl" scale="${mesh_scale} ${mesh_scale} ${mesh_scale}"/>
             </geometry>
-            <material name="arm_material"/>
-            <!--
+            <material name="arm_material"/> -->
             <origin xyz="-0.035 0 0" rpy="0 0 0"/>
             <geometry>
                 <box size="0.09 0.025 0.035" />
             </geometry>
-            -->
         </collision>
         <visual>
@@ -59,15 +57,13 @@
         </xacro:inertial_box>
         <collision>
-            <origin xyz="-0.02 0.05 0" rpy="${pi/2} 0 0"/>
+            <!-- <origin xyz="-0.02 0.05 0" rpy="${pi/2} 0 0"/>
             <geometry>
                 <mesh filename="${mesh_folder}version_6/arm_v2/arm_segment_1_reduced.stl" scale="${mesh_scale} ${mesh_scale} ${mesh_scale}"/>
             </geometry>
-            <material name="arm_material"/>
-            <!--
+            <material name="arm_material"/> -->
             <origin xyz="-0.02 0.025 0" rpy="0 0 0"/>
             <geometry>
                 <box size="0.025 0.075 0.035" />
             </geometry>
-            -->
         </collision>
         <visual>
@@ -91,15 +87,13 @@
         </xacro:inertial_box>
         <collision>
-            <origin xyz="0 0 0" rpy="${-pi/2} 0 0"/>
+            <!-- <origin xyz="0 0 0" rpy="${-pi/2} 0 0"/>
             <geometry>
                 <mesh filename="${mesh_folder}version_6/arm_v2/arm_segment_2_reduced.stl" scale="${mesh_scale} ${mesh_scale} ${mesh_scale}"/>
             </geometry>
-            <material name="arm_material"/>
-            <!--
+            <material name="arm_material"/> -->
             <origin xyz="0.045 0 0" rpy="0 0 0"/>
             <geometry>
                 <box size="0.05 0.03 0.035" />
             </geometry>
-            -->
         </collision>
         <visual>

File: config/urdf/version_6/chassis.xacro (robot description, xacro)
@@ -15,5 +15,5 @@
             <origin xyz="0 0 -0.005" rpy="0 0 0"/>
         </xacro:inertial_box>
-        <!-- <collision>
+        <collision>
             <origin xyz="0 0 -0.005" rpy="0 0 0"/>
             <geometry>
@@ -26,6 +26,6 @@
                 <box size="0.13 0.16 0.06" />
             </geometry>
-        </collision> -->
-        <collision>
+        </collision>
+        <!-- <collision>
             <origin xyz="0 0 0" rpy="0 0 0"/>
             <geometry>
@@ -33,5 +33,5 @@
             </geometry>
             <material name="chassis_material"/>
-        </collision>
+        </collision> -->
         <visual>
             <origin xyz="0 0 0" rpy="0 0 0"/>

File: config/urdf/version_6/gripper.xacro (robot description, xacro)
@@ -19,5 +19,5 @@
         <origin xyz="-0.0207 0.0125 0.0355" rpy="0 0 0"/>
         <axis xyz="0 0 1" />
-        <limit lower="0" upper="0" velocity="0" effort="0"/>
+        <limit lower="0" upper="1.7" velocity="0" effort="0"/>
     </joint>
     <link name="gripper_link">
@@ -61,5 +61,5 @@
                 <material name="gripper_material"/>
             </visual>
-            <collision>
+            <!-- <collision>
                 <origin xyz="0 0 0" rpy="0 0 ${pi/2+multiplier*pi/2}"/>
                 <geometry>
@@ -67,5 +67,5 @@
                 </geometry>
                 <material name="gripper_material"/>
-            </collision>
+            </collision> -->
         </link>
         <joint name="gripper_${side}_front_piece_joint" type="continuous">
@@ -89,5 +89,5 @@
                 <material name="gripper_material"/>
             </visual>
-            <collision>
+            <!-- <collision>
                 <origin xyz="0 0 0" rpy="0 0 ${pi/2+multiplier*pi/2}"/>
                 <geometry>
@@ -95,5 +95,5 @@
                 </geometry>
                 <material name="gripper_material"/>
-            </collision>
+            </collision> -->
         </link>
         <joint name="gripper_${side}_joint" type="continuous">
@@ -117,5 +117,5 @@
                 <material name="gripper_material"/>
             </visual>
-            <collision>
+            <!-- <collision>
                 <origin xyz="0 0 0" rpy="0 0 0"/>
                 <geometry>
@@ -123,5 +123,5 @@
                 </geometry>
                 <material name="gripper_material"/>
-            </collision>
+            </collision> -->
         </link>
     </xacro:macro>

File: config/urdf/version_6/wheels.xacro (robot description, xacro)
@@ -20,15 +20,13 @@
             </visual>
             <collision>
-                <origin xyz="0 0 0" rpy="${visual_rpy}"/>
+                <!-- <origin xyz="0 0 0" rpy="${visual_rpy}"/>
                 <geometry>
                     <mesh filename="${mesh_folder}version_6/wheel_reduced.stl" scale="${mesh_scale} ${mesh_scale} ${mesh_scale}"/>
                 </geometry>
-                <material name="wheel_material"/>
-                <!--
+                <material name="wheel_material"/> -->
                 <origin xyz="${collision_xyz}" rpy="${pi/2} 0 0"/>
                 <geometry>
                     <cylinder radius="0.06" length="0.04" />
                 </geometry>
-                -->
                 <surface>
                     <friction>
@@ -48,5 +46,5 @@
     <xacro:wheel name="wheel_front_left" xyz="0.109 0.063 -0.079" visual_rpy="0 0 ${pi}" collision_xyz="0 0.03 0" />
     <xacro:wheel name="wheel_front_right" xyz="0.109 -0.063 -0.079" visual_rpy="0 0 0" collision_xyz="0 -0.03 0" />
-    <xacro:wheel name="wheel_rear_left" xyz="-0.109 0.063 -0.079" visual_rpy="0 0 ${pi}" collision_xyz="0 0.03 0" />
-    <xacro:wheel name="wheel_rear_right" xyz="-0.109 -0.063 -0.079" visual_rpy="0 0 0" collision_xyz="0 -0.03 0" />
+    <xacro:wheel name="wheel_back_left" xyz="-0.109 0.063 -0.079" visual_rpy="0 0 ${pi}" collision_xyz="0 0.03 0" />
+    <xacro:wheel name="wheel_back_right" xyz="-0.109 -0.063 -0.079" visual_rpy="0 0 0" collision_xyz="0 -0.03 0" />
 </robot>
