Commit message: mujoco + better urdf compilation

File: config/urdf/d435.xacro (robot description, xacro)
@@ -67,5 +67,5 @@
         <origin xyz="${d435_zero_depth_to_glass + d435_glass_to_front} ${-d435_cam_depth_py} 0" rpy="${M_PI/2} 0 ${M_PI/2}"/>
         <geometry>
-          <mesh filename="package://quac/meshes/d435.dae" />
+          <mesh filename="${mesh_folder}d435.dae" />
         </geometry>
         <material name="aluminum" />

File: config/urdf/oak_d_lite.xacro (robot description, xacro)
@@ -18,8 +18,15 @@
 				<origin xyz="0 0 0" rpy="0 0 0" />
 				<geometry>
-					<mesh filename="package://quac/meshes/oak_d_lite.stl" />
+					<mesh filename="${mesh_folder}oak_d_lite.stl" />
 				</geometry>
 				<material name="oak_d_lite_material"/>
 			</visual>
+			<collision>
+				<origin xyz="0 0 0" rpy="0 0 0" />
+				<geometry>
+					<mesh filename="${mesh_folder}oak_d_lite.stl" />
+				</geometry>
+				<material name="oak_d_lite_material"/>
+			</collision>
 		</link>
 		<joint name="${camera_name}_model_origin_joint" type="fixed">

File: config/urdf/robot.urdf.xacro (robot description, xacro)
@@ -2,4 +2,6 @@
 <robot xmlns:xacro="http://www.ros.org/wiki/xacro"  name="quac_robot">
     <xacro:property name="mesh_scale" value="1"/>
+    <xacro:arg name="mesh_folder" default="mesh_folder_path/"/>
+    <xacro:property name="mesh_folder" value="$(arg mesh_folder)"/>
     <xacro:include filename="inertial_macros.xacro" />
     <xacro:include filename="servo.xacro" />

File: config/urdf/version_6/arm_v2.xacro (robot description, xacro)
@@ -11,9 +11,7 @@
     </joint>
     <link name="arm_base_link">
-        <inertial>
+        <xacro:inertial_box mass="0.1" x="0.01" y="0.01" z="0.01">
             <origin xyz="0 0 0" rpy="0 0 0"/>
-            <mass value="0.1"/>
-            <inertia ixx="0.01" ixy="0.0" ixz="0.0" iyy="0.01" iyz="0.0" izz="0.01"/>
-        </inertial>
+        </xacro:inertial_box>
     </link>
     <joint name="arm_segment_0_joint" type="revolute">
@@ -25,13 +23,24 @@
     </joint>
     <link name="arm_segment_0">
-        <inertial>
-            <origin xyz="0 0 0" rpy="0 0 0"/>
-            <mass value="0.2"/>
-            <inertia ixx="0.01" ixy="0.0" ixz="0.0" iyy="0.01" iyz="0.0" izz="0.01"/>
-        </inertial>
+        <xacro:inertial_box mass="0.15" x="0.09" y="0.025" z="0.035">
+            <origin xyz="-0.035 0 0" rpy="0 0 0"/>
+        </xacro:inertial_box>
+        <collision>
+            <origin xyz="0 0 0" rpy="${-pi/2} 0 0"/>
+            <geometry>
+                <mesh filename="${mesh_folder}version_6/arm_v2/arm_segment_0_reduced.stl" scale="${mesh_scale} ${mesh_scale} ${mesh_scale}"/>
+            </geometry>
+            <material name="arm_material"/>
+            <!--
+            <origin xyz="-0.035 0 0" rpy="0 0 0"/>
+            <geometry>
+                <box size="0.09 0.025 0.035" />
+            </geometry>
+            -->
+        </collision>
         <visual>
             <origin xyz="0 0 0" rpy="${-pi/2} 0 0"/>
             <geometry>
-                <mesh filename="package://quac/meshes/version_6/arm_v2/arm_segment_0_reduced.stl" scale="${mesh_scale} ${mesh_scale} ${mesh_scale}"/>
+                <mesh filename="${mesh_folder}version_6/arm_v2/arm_segment_0_reduced.stl" scale="${mesh_scale} ${mesh_scale} ${mesh_scale}"/>
             </geometry>
             <material name="arm_material"/>
@@ -46,13 +55,24 @@
     </joint>
     <link name="arm_segment_1">
-        <inertial>
-            <origin xyz="0 0 0" rpy="0 0 0"/>
-            <mass value="0.2"/>
-            <inertia ixx="0.01" ixy="0.0" ixz="0.0" iyy="0.01" iyz="0.0" izz="0.01"/>
-        </inertial>
+        <xacro:inertial_box mass="0.1" x="0.025" y="0.075" z="0.035">
+            <origin xyz="-0.02 0.025 0" rpy="0 0 0"/>
+        </xacro:inertial_box>
+        <collision>
+            <origin xyz="-0.02 0.05 0" rpy="${pi/2} 0 0"/>
+            <geometry>
+                <mesh filename="${mesh_folder}version_6/arm_v2/arm_segment_1_reduced.stl" scale="${mesh_scale} ${mesh_scale} ${mesh_scale}"/>
+            </geometry>
+            <material name="arm_material"/>
+            <!--
+            <origin xyz="-0.02 0.025 0" rpy="0 0 0"/>
+            <geometry>
+                <box size="0.025 0.075 0.035" />
+            </geometry>
+            -->
+        </collision>
         <visual>
             <origin xyz="-0.02 0.05 0" rpy="${pi/2} 0 0"/>
             <geometry>
-                <mesh filename="package://quac/meshes/version_6/arm_v2/arm_segment_1_reduced.stl" scale="${mesh_scale} ${mesh_scale} ${mesh_scale}"/>
+                <mesh filename="${mesh_folder}version_6/arm_v2/arm_segment_1_reduced.stl" scale="${mesh_scale} ${mesh_scale} ${mesh_scale}"/>
             </geometry>
             <material name="arm_material"/>
@@ -67,13 +87,24 @@
     </joint>
     <link name="arm_segment_2">
-        <inertial>
-            <origin xyz="0 0 0" rpy="0 0 0"/>
-            <mass value="0.2"/>
-            <inertia ixx="0.01" ixy="0.0" ixz="0.0" iyy="0.01" iyz="0.0" izz="0.01"/>
-        </inertial>
+        <xacro:inertial_box mass="0.05" x="0.05" y="0.03" z="0.035">
+            <origin xyz="0.045 0 0" rpy="0 0 0"/>
+        </xacro:inertial_box>
+        <collision>
+            <origin xyz="0 0 0" rpy="${-pi/2} 0 0"/>
+            <geometry>
+                <mesh filename="${mesh_folder}version_6/arm_v2/arm_segment_2_reduced.stl" scale="${mesh_scale} ${mesh_scale} ${mesh_scale}"/>
+            </geometry>
+            <material name="arm_material"/>
+            <!--
+            <origin xyz="0.045 0 0" rpy="0 0 0"/>
+            <geometry>
+                <box size="0.05 0.03 0.035" />
+            </geometry>
+            -->
+        </collision>
         <visual>
             <origin xyz="0 0 0" rpy="${-pi/2} 0 0"/>
             <geometry>
-                <mesh filename="package://quac/meshes/version_6/arm_v2/arm_segment_2_reduced.stl" scale="${mesh_scale} ${mesh_scale} ${mesh_scale}"/>
+                <mesh filename="${mesh_folder}version_6/arm_v2/arm_segment_2_reduced.stl" scale="${mesh_scale} ${mesh_scale} ${mesh_scale}"/>
             </geometry>
             <material name="arm_material"/>

File: config/urdf/version_6/chassis.xacro (robot description, xacro)
@@ -12,13 +12,30 @@
     </joint>
     <link name="chassis">
-        <inertial>
-            <origin xyz="-0.006592503505638408 -1.5301626995551604e-17 0.04294027543409115" rpy="0 0 0"/>
-            <mass value="6.419279977222798"/>
-            <inertia ixx="0.031932" iyy="0.058111" izz="0.057234" ixy="-0.0" iyz="-0.0" ixz="0.003075"/>
-        </inertial>
+        <xacro:inertial_box mass="2.5" x="0.31" y="0.12" z="0.07">
+            <origin xyz="0 0 -0.005" rpy="0 0 0"/>
+        </xacro:inertial_box>
+        <!-- <collision>
+            <origin xyz="0 0 -0.005" rpy="0 0 0"/>
+            <geometry>
+                <box size="0.31 0.12 0.07" />
+            </geometry>
+        </collision>
+        <collision>
+            <origin xyz="-0.055 0 0.06" rpy="0 0 0"/>
+            <geometry>
+                <box size="0.13 0.16 0.06" />
+            </geometry>
+        </collision> -->
+        <collision>
+            <origin xyz="0 0 0" rpy="0 0 0"/>
+            <geometry>
+                <mesh filename="${mesh_folder}version_6/chassis_reduced.stl" scale="${mesh_scale} ${mesh_scale} ${mesh_scale}"/>
+            </geometry>
+            <material name="chassis_material"/>
+        </collision>
         <visual>
             <origin xyz="0 0 0" rpy="0 0 0"/>
             <geometry>
-                <mesh filename="package://quac/meshes/version_6/chassis_reduced.stl" scale="${mesh_scale} ${mesh_scale} ${mesh_scale}"/>
+                <mesh filename="${mesh_folder}version_6/chassis_reduced.stl" scale="${mesh_scale} ${mesh_scale} ${mesh_scale}"/>
             </geometry>
             <material name="chassis_material"/>

File: config/urdf/version_6/gripper.xacro (robot description, xacro)
@@ -8,5 +8,5 @@
             <origin xyz="0 0 0" rpy="0 0 0"/>
             <mass value="0.1"/>
-            <inertia ixx="0.01" ixy="0.0" ixz="0.0" iyy="0.01" iyz="0.0" izz="0.01"/>
+            <inertia ixx="0.001" ixy="0.0" ixz="0.0" iyy="0.001" iyz="0.0" izz="0.001"/>
         </inertial>
     </link>
@@ -25,5 +25,5 @@
             <origin xyz="0 0 0" rpy="0 0 0"/>
             <mass value="0.1"/>
-            <inertia ixx="0.01" ixy="0.0" ixz="0.0" iyy="0.01" iyz="0.0" izz="0.01"/>
+            <inertia ixx="0.001" ixy="0.0" ixz="0.0" iyy="0.001" iyz="0.0" izz="0.001"/>
         </inertial>
     </link>
@@ -57,8 +57,15 @@
                 <origin xyz="0 0 0" rpy="0 0 ${pi/2+multiplier*pi/2}"/>
                 <geometry>
-                    <mesh filename="package://quac/meshes/version_6/gripper_back_piece.stl" scale="${mesh_scale} ${mesh_scale} ${mesh_scale}"/>
+                    <mesh filename="${mesh_folder}version_6/gripper_back_piece.stl" scale="${mesh_scale} ${mesh_scale} ${mesh_scale}"/>
                 </geometry>
                 <material name="gripper_material"/>
             </visual>
+            <collision>
+                <origin xyz="0 0 0" rpy="0 0 ${pi/2+multiplier*pi/2}"/>
+                <geometry>
+                    <mesh filename="${mesh_folder}version_6/gripper_back_piece.stl" scale="${mesh_scale} ${mesh_scale} ${mesh_scale}"/>
+                </geometry>
+                <material name="gripper_material"/>
+            </collision>
         </link>
         <joint name="gripper_${side}_front_piece_joint" type="continuous">
@@ -78,8 +85,15 @@
                 <origin xyz="0 0 0" rpy="0 0 ${pi/2+multiplier*pi/2}"/>
                 <geometry>
-                    <mesh filename="package://quac/meshes/version_6/gripper_front_piece.stl" scale="${mesh_scale} ${mesh_scale} ${mesh_scale}"/>
+                    <mesh filename="${mesh_folder}version_6/gripper_front_piece.stl" scale="${mesh_scale} ${mesh_scale} ${mesh_scale}"/>
                 </geometry>
                 <material name="gripper_material"/>
             </visual>
+            <collision>
+                <origin xyz="0 0 0" rpy="0 0 ${pi/2+multiplier*pi/2}"/>
+                <geometry>
+                    <mesh filename="${mesh_folder}version_6/gripper_front_piece.stl" scale="${mesh_scale} ${mesh_scale} ${mesh_scale}"/>
+                </geometry>
+                <material name="gripper_material"/>
+            </collision>
         </link>
         <joint name="gripper_${side}_joint" type="continuous">
@@ -99,8 +113,15 @@
                 <origin xyz="0 0 0" rpy="0 0 0"/>
                 <geometry>
-                    <mesh filename="package://quac/meshes/version_6/gripper_${side}.stl" scale="${mesh_scale} ${mesh_scale} ${mesh_scale}"/>
+                    <mesh filename="${mesh_folder}version_6/gripper_${side}.stl" scale="${mesh_scale} ${mesh_scale} ${mesh_scale}"/>
                 </geometry>
                 <material name="gripper_material"/>
             </visual>
+            <collision>
+                <origin xyz="0 0 0" rpy="0 0 0"/>
+                <geometry>
+                    <mesh filename="${mesh_folder}version_6/gripper_${side}.stl" scale="${mesh_scale} ${mesh_scale} ${mesh_scale}"/>
+                </geometry>
+                <material name="gripper_material"/>
+            </collision>
         </link>
     </xacro:macro>

File: config/urdf/version_6/wheels.xacro (robot description, xacro)
@@ -15,13 +15,20 @@
                 <origin xyz="0 0 0" rpy="${visual_rpy}"/>
                 <geometry>
-                    <mesh filename="package://quac/meshes/version_6/wheel_reduced.stl" scale="${mesh_scale} ${mesh_scale} ${mesh_scale}"/>
+                    <mesh filename="${mesh_folder}version_6/wheel_reduced.stl" scale="${mesh_scale} ${mesh_scale} ${mesh_scale}"/>
                 </geometry>
                 <material name="wheel_material"/>
             </visual>
             <collision>
+                <origin xyz="0 0 0" rpy="${visual_rpy}"/>
+                <geometry>
+                    <mesh filename="${mesh_folder}version_6/wheel_reduced.stl" scale="${mesh_scale} ${mesh_scale} ${mesh_scale}"/>
+                </geometry>
+                <material name="wheel_material"/>
+                <!--
                 <origin xyz="${collision_xyz}" rpy="${pi/2} 0 0"/>
                 <geometry>
                     <cylinder radius="0.06" length="0.04" />
                 </geometry>
+                -->
                 <surface>
                     <friction>

Commit message: mujoco general functionality + redid config

File: config/urdf/d435.xacro (robot description, xacro)
@@ -29,6 +29,6 @@
     <!-- The following values are approximate, and the camera node
      publishing TF values with actual calibrated camera extrinsic values -->
-    <xacro:property name="d435_cam_depth_to_infra1_offset" value="0.0"/>
-    <xacro:property name="d435_cam_depth_to_infra2_offset" value="-0.050"/>
+    <xacro:property name="d435_cam_depth_to_stereo_left_offset" value="0.0"/>
+    <xacro:property name="d435_cam_depth_to_stereo_right_offset" value="-0.050"/>
     <xacro:property name="d435_cam_depth_to_color_offset" value="0.015"/>
     <!-- The following values model the aluminum peripherial case for the
@@ -100,29 +100,29 @@
       <link name="${name}_depth_optical_frame"/>
       <!-- camera left IR joints and links -->
-      <joint name="${name}_infra1_joint" type="fixed">
-        <origin xyz="0 ${d435_cam_depth_to_infra1_offset} 0" rpy="0 0 0" />
+      <joint name="${name}_stereo_left_joint" type="fixed">
+        <origin xyz="0 ${d435_cam_depth_to_stereo_left_offset} 0" rpy="0 0 0" />
         <parent link="${name}_link" />
-        <child link="${name}_infra1_frame" />
+        <child link="${name}_stereo_left_frame" />
       </joint>
-      <link name="${name}_infra1_frame"/>
-      <joint name="${name}_infra1_optical_joint" type="fixed">
+      <link name="${name}_stereo_left_frame"/>
+      <joint name="${name}_stereo_left_optical_joint" type="fixed">
         <origin xyz="0 0 0" rpy="${-M_PI/2} 0 ${-M_PI/2}" />
-        <parent link="${name}_infra1_frame" />
-        <child link="${name}_infra1_optical_frame" />
+        <parent link="${name}_stereo_left_frame" />
+        <child link="${name}_stereo_left_optical_frame" />
       </joint>
-      <link name="${name}_infra1_optical_frame"/>
+      <link name="${name}_stereo_left_optical_frame"/>
       <!-- camera right IR joints and links -->
-      <joint name="${name}_infra2_joint" type="fixed">
-        <origin xyz="0 ${d435_cam_depth_to_infra2_offset} 0" rpy="0 0 0" />
+      <joint name="${name}_stereo_right_joint" type="fixed">
+        <origin xyz="0 ${d435_cam_depth_to_stereo_right_offset} 0" rpy="0 0 0" />
         <parent link="${name}_link" />
-        <child link="${name}_infra2_frame" />
+        <child link="${name}_stereo_right_frame" />
       </joint>
-      <link name="${name}_infra2_frame"/>
-      <joint name="${name}_infra2_optical_joint" type="fixed">
+      <link name="${name}_stereo_right_frame"/>
+      <joint name="${name}_stereo_right_optical_joint" type="fixed">
         <origin xyz="0 0 0" rpy="${-M_PI/2} 0 ${-M_PI/2}" />
-        <parent link="${name}_infra2_frame" />
-        <child link="${name}_infra2_optical_frame" />
+        <parent link="${name}_stereo_right_frame" />
+        <child link="${name}_stereo_right_optical_frame" />
       </joint>
-      <link name="${name}_infra2_optical_frame"/>
+      <link name="${name}_stereo_right_optical_frame"/>
       <!-- camera color joints and links -->
       <joint name="${name}_color_joint" type="fixed">

File: config/urdf/oak_d_lite.xacro (robot description, xacro)
@@ -6,6 +6,6 @@
 	<xacro:macro name="oak_d_lite" params="camera_name parent xyz rpy">
 		<xacro:property name="baseline" value="0.075" />
-		<xacro:property name="left_name" value="infra2" />
-		<xacro:property name="right_name" value="infra1" />
+		<xacro:property name="left_name" value="stereo_right" />
+		<xacro:property name="right_name" value="stereo_left" />
 		<link name="${camera_name}" />
 		<joint name="${camera_name}_center_joint" type="fixed">
